File: Hardware/apr-sensor/apr-sensor.kicad_sch (KiCad schematic)
At the start: 43 parts, among them J1 Conn_02x05_Odd_Even, J2 Micro_SD_Card, J3 Conn_01x02_Male, J4 Conn_01x02_Male, J5 Conn_01x02_Male, J6 Conn_Coaxial, U1 ATSAMD21E17D-M, U2 LSM6DSO32TR, U3 RockBLOCK-9603, U4 MTK3339

Commit message: APR-Sensor Floorplanning
Parts:
- removed J4: Conn_01x02_Male, symbol Connector:Conn_01x02_Male
- removed U4: MTK3339, symbol GQC:MTK3339
- added C7, C8: 100n, Capacitor_SMD:C_0603_1608Metric, symbol Device:C_Small
- added D3: D_TVS_Filled, Diode_SMD:D_0201_0603Metric, symbol Device:D_TVS_Filled
- added FB2: FerriteBead_Small, Inductor_SMD:L_0603_1608Metric, symbol Device:FerriteBead_Small
- added G1: GQC-Logo, GQC:GQC-Logo, symbol GQC:GQC-Logo
- added J4: USB_B_Mini, Connector_USB:USB_Mini-B_Wuerth_65100516121_Horizontal, symbol Connector:USB_B_Mini
- added J7: Conn_01x02_Male, Connector_PinHeader_2.54mm:PinHeader_1x02_P2.54mm_Vertical, symbol Connector:Conn_01x02_Male
- added U4: PA1616S, GQC:FGPMMOPA6H, symbol GQC:PA1616S
- added U5: MCP1793T-3302H-DC, Package_TO_SOT_SMD:SOT-223-6, symbol GQC:MCP1793T-3302H-DC
- C1, C2, C3, C4, C5, C6: footprint (none) -> Capacitor_SMD:C_0603_1608Metric
- D1, D2: footprint (none) -> LED_SMD:LED_0805_2012Metric
- FB1: footprint (none) -> Inductor_SMD:L_0603_1608Metric
- J1: footprint (none) -> GQC:3221-10-0300-00-TR
- J3, J5: footprint (none) -> Connector_PinHeader_2.54mm:PinHeader_1x02_P2.54mm_Vertical
- J6: footprint (none) -> Connector_Coaxial:SMA_Samtec_SMA-J-P-X-ST-EM1_EdgeMount
- R1, R2: footprint (none) -> Resistor_SMD:R_0603_1608Metric
- TP1, TP10, TP11, TP12, TP13, TP14, TP15, TP16, TP17, TP18, TP19, TP2, TP20, TP21, TP22, TP3, TP4, TP5, TP6, TP7, TP8, TP9: footprint (none) -> GQC:RCU-0603
- U3: footprint (none) -> Connector_Molex:Molex_PicoBlade_53047-1010_1x10_P1.25mm_Vertical
Connections:
- net +3V3: now also J7.1 (Pin_1), U4.1 (VCC)
- net +5V: now also C7.2, D3.2 (A2), FB2.2, U5.1 (~{SHDN}), U5.2 (VIN)
- net GND: now also C7.1, C8.1, D3.1 (A1), J4.5 (GND), J4.6 (Shield), U4. (GND), U4.12 (GND), U4.19 (GND), U4.3 (GND), U4.8 (GND), U5.3 (GND), U5.6 (GND)
- net GPS_1PPS: now also U4.13 (1PPS); no longer TP13.1, U1.15 (PA14)
- net GPS_FIX: now also TP13.1, U1.15 (PA14), U4.5 (3D-FIX)
- net GPS_~{RST}: now also U4.2 (~{RST})
- net SC3_RXD: now also U4.9 (TX)
- net SC3_TXD: now also U4.10 (RX)
- net at J6.1 (In): now also U4.11 (EX_ANT)
- net at J5.1 (Pin_1): now also U4.4 (VBKUP)
- new net: C8.2, J7.2 (Pin_2), U5.4 (VOUT)
- new net: FB2.1, J4.1 (VBUS)
- no-connect marks 9 -> 12
Other:
- moved on the sheet: J3
