File: Hardware/aatr-sensor/aatr-sensor.kicad_sch (KiCad schematic)
At the start: 50 parts, among them J1 Conn_02x05_Odd_Even, J2 Micro_SD_Card, J3 Conn_01x02_Male, J4 USB_B_Mini, J5 Conn_01x02_Male, J6 Conn_Coaxial, J7 Conn_01x02_Male, U1 ATSAMD21E17D-M, U2 LSM6DSO32TR, U3 RockBLOCK-9603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

Commit message: AATR-Sensor: Create BOM, CAM Files
Parts:
- J4: footprint Connector_USB:USB_Mini-B_Wuerth_65100516121_Horizontal -> GQC:USB_Mini-B_Wuerth_65100516121_Horizontal
- J6: footprint Connector_Coaxial:SMA_Samtec_SMA-J-P-X-ST-EM1_EdgeMount -> GQC:SMA_Samtec_SMA-J-P-X-ST-EM1_EdgeMount
- U3: footprint Connector_Molex:Molex_PicoBlade_53047-1010_1x10_P1.25mm_Vertical -> GQC:Molex_PicoBlade_53047-1010_1x10_P1.25mm_Vertical
- U5: footprint Package_TO_SOT_SMD:SOT-223-6 -> GQC:SOT-223-6
Changed lines of the file:
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@@
     (property "Reference" "J4" (id 0) (at 144.78 15.24 0))
     (property "Value" "USB_B_Mini" (id 1) (at 144.78 17.78 0))
-    (property "Footprint" "Connector_USB:USB_Mini-B_Wuerth_65100516121_Horizontal" (id 2) (at 148.59 27.94 0)
+    (property "Footprint" "GQC:USB_Mini-B_Wuerth_65100516121_Horizontal" (id 2) (at 148.59 27.94 0)
       (effects (font (size 1.27 1.27)) hide)
     )
@@
     (property "Reference" "U5" (id 0) (at 209.55 17.78 0))
     (property "Value" "MCP1793T-3302H-DC" (id 1) (at 209.55 20.32 0))
-    (property "Footprint" "Package_TO_SOT_SMD:SOT-223-6" (id 2) (at 201.93 24.13 0)
+    (property "Footprint" "GQC:SOT-223-6" (id 2) (at 201.93 24.13 0)
       (effects (font (size 1.27 1.27)) hide)
     )
@@
       (effects (font (size 1.27 1.27)) (justify left))
     )
-    (property "Footprint" "Connector_Coaxial:SMA_Samtec_SMA-J-P-X-ST-EM1_EdgeMount" (id 2) (at 255.27 129.54 0)
+    (property "Footprint" "GQC:SMA_Samtec_SMA-J-P-X-ST-EM1_EdgeMount" (id 2) (at 255.27 129.54 0)
       (effects (font (size 1.27 1.27)) hide)
     )
@@
       (effects (font (size 1.27 1.27)) (justify left))
     )
-    (property "Footprint" "Connector_Molex:Molex_PicoBlade_53047-1010_1x10_P1.25mm_Vertical" (id 2) (at 219.71 66.04 0)
+    (property "Footprint" "GQC:Molex_PicoBlade_53047-1010_1x10_P1.25mm_Vertical" (id 2) (at 219.71 66.04 0)
       (effects (font (size 1.27 1.27)) hide)
     )
@@
     )
     (path "/bdaf8834-d2f5-4491-a90e-52fe9d0565ca"
-      (reference "J4") (unit 1) (value "USB_B_Mini") (footprint "Connector_USB:USB_Mini-B_Wuerth_65100516121_Horizontal")
+      (reference "J4") (unit 1) (value "USB_B_Mini") (footprint "GQC:USB_Mini-B_Wuerth_65100516121_Horizontal")
     )
     (path "/b7eafe31-f653-4d63-ab31-f880d6d43277"
@@
     )
     (path "/f0b8cf79-8c57-480a-b337-db4b2a375dfa"
-      (reference "J6") (unit 1) (value "Conn_Coaxial") (footprint "Connector_Coaxial:SMA_Samtec_SMA-J-P-X-ST-EM1_EdgeMount")
+      (reference "J6") (unit 1) (value "Conn_Coaxial") (footprint "GQC:SMA_Samtec_SMA-J-P-X-ST-EM1_EdgeMount")
     )
     (path "/121f28a8-4d1a-4067-8479-a7d9be548c12"
@@
     )
     (path "/f4400a84-e131-4565-87f8-21512e77e8d4"
-      (reference "U3") (unit 1) (value "RockBLOCK-9603") (footprint "Connector_Molex:Molex_PicoBlade_53047-1010_1x10_P1.25mm_Vertical")
+      (reference "U3") (unit 1) (value "RockBLOCK-9603") (footprint "GQC:Molex_PicoBlade_53047-1010_1x10_P1.25mm_Vertical")
     )
     (path "/0c101c6e-8c71-47ea-ac80-64dc2a6fa2d1"
@@
     )
     (path "/e3905afb-f595-419b-bf7d-21c586978025"
-      (reference "U5") (unit 1) (value "MCP1793T-3302H-DC") (footprint "Package_TO_SOT_SMD:SOT-223-6")
-    )
-  )
+      (reference "U5") (unit 1) (value "MCP1793T-3302H-DC") (footprint "GQC:SOT-223-6")
+    )
+  )
